Commit message: Add dockerfile

File: tasks/models/urdf/iiwa_airhockey.urdf (robot description, URDF)
Before this commit: robot iiwa_1, 15 links, 14 joints
Links:
- removed link world
- added link base_link
- link iiwa_1/link_4: geometry collision mesh filename=meshes/iiwa_airhockey/collision/link_4.stl; visual mesh filename=meshes/iiwa_airhockey/visual/link_4.stl
Joints:
- joint iiwa_1/base_joint: parent world -> base_link
