Commit message: Add dockerfile and and new env

File: tasks/models/urdf/airhockey_table.urdf (robot description, URDF)
Before this commit: robot airhockey_table, 1 links, 0 joints
Links:
- link baseLink: geometry collision box size=0.3 0.3 0.2; collision mesh filename=meshes/iiwa_airhockey/table/table.stl scale=0.1 0.1 0.58

Commit message: Update scenes

File: tasks/models/urdf/airhockey_table.urdf (robot description, URDF)
Before this commit: robot airhockey_table, 1 links, 0 joints
Links:
- link baseLink: geometry collision box size=2 1.2 0.1; visual mesh filename=meshes/iiwa_airhockey/table/table.dae

File: tasks/models/urdf/block.urdf (robot description, URDF)
Before this commit: robot block, 1 links, 0 joints
Links:
- link baseLink: geometry collision box size=0.2 0.3 0.02; visual box size=0.2 0.3 0.075

File: tasks/models/urdf/peg_round.urdf (robot description, URDF)
Before this commit: robot peg_round, 2 links, 1 joints
Links:
- link peg_link: geometry visual mesh filename=meshes/peg/peg_round.STL scale=0.001 0.001 0.001
