Commit message: Fix scene for ffual arm

File: tasks/models/urdf/table.urdf (robot description, URDF)
Before this commit: robot table.urdf, 1 links, 0 joints
Links:
- link baseLink: geometry collision box size=1.5 1.2 0.05; visual mesh filename=meshes/table/table.obj scale=0.1 0.1 0.58

File: tasks/models/urdf/ur5e_pybullet.urdf (robot description, URDF)
Before this commit: robot ur5e, 13 links, 12 joints
Links:
- link base_link: geometry collision mesh filename=meshes/ur5e/collision/base.stl; visual mesh filename=meshes/ur5e/visual/base.obj
- link forearm_link: geometry collision mesh filename=meshes/ur5e/collision/forearm.stl; visual mesh filename=meshes/ur5e/visual/forearm.obj
- link shoulder_link: geometry collision mesh filename=meshes/ur5e/collision/shoulder.stl; visual mesh filename=meshes/ur5e/visual/shoulder.obj
- link upper_arm_link: geometry collision mesh filename=meshes/ur5e/collision/upperarm.stl; visual mesh filename=meshes/ur5e/visual/upperarm.obj
- link wrist_1_link: geometry collision mesh filename=meshes/ur5e/collision/wrist1.stl; visual mesh filename=meshes/ur5e/visual/wrist1.obj
- link wrist_2_link: geometry collision mesh filename=meshes/ur5e/collision/wrist2.stl; visual mesh filename=meshes/ur5e/visual/wrist2.obj
- link wrist_3_link: geometry collision mesh filename=meshes/ur5e/collision/wrist3.stl; visual mesh filename=meshes/ur5e/visual/wrist3.obj

File: tasks/models/urdf/ur5e_pybullet2.urdf (robot description, URDF)
Before this commit: robot ur5e, 13 links, 12 joints
Links:
- link base_link: geometry collision mesh filename=meshes/ur5e/collision/base.stl; visual mesh filename=meshes/ur5e/visual/base.obj
- link forearm_link: geometry collision mesh filename=meshes/ur5e/collision/forearm.stl; visual mesh filename=meshes/ur5e/visual/forearm.obj
- link shoulder_link: geometry collision mesh filename=meshes/ur5e/collision/shoulder.stl; visual mesh filename=meshes/ur5e/visual/shoulder.obj
- link upper_arm_link: geometry collision mesh filename=meshes/ur5e/collision/upperarm.stl; visual mesh filename=meshes/ur5e/visual/upperarm.obj
- link wrist_1_link: geometry collision mesh filename=meshes/ur5e/collision/wrist1.stl; visual mesh filename=meshes/ur5e/visual/wrist1.obj
- link wrist_2_link: geometry collision mesh filename=meshes/ur5e/collision/wrist2.stl; visual mesh filename=meshes/ur5e/visual/wrist2.obj
- link wrist_3_link: geometry collision mesh filename=meshes/ur5e/collision/wrist3.stl; visual mesh filename=meshes/ur5e/visual/wrist3.obj
Joints:
- joint base-base_link_fixed_joint: origin xyz=0 0 0 rpy=0 0 0.0 -> xyz=0 0 0 rpy=0 0 0
